Commit message: update robot definition

File: src/my_robot/urdf/my_robot.xacro (robot description, xacro)
@@ -35,7 +35,4 @@
     <dynamics damping="1.0" friction="1.0"/>
   </joint>
-  <gazebo reference="left_wheel">
-    <material>Gazebo/Black</material>
-  </gazebo>
     <link name="right_wheel">
       <inertial>
@@ -61,7 +58,4 @@
 	</visual>
     </link>
-  <gazebo reference="right_wheel">
-    <material>Gazebo/Black</material>
-  </gazebo>
   <joint type="continuous" name="right_wheel_hinge">
     <origin xyz="0 -0.230 0" rpy="0 0 0"/>
@@ -72,13 +66,14 @@
     <dynamics damping="1.0" friction="1.0"/>
   </joint>
-   <link name="camera_plate">
-       <pose>0 0 0.3 0 0 0</pose>
+   <!-- Camera platform -->
+   <link name="camera_platform">
+       <pose>0 0 0 0 0 0</pose>
     <inertial>
-      <mass value="15.0"/>
-      <origin xyz="0.0 0 0" rpy=" 0 0 0"/>
-      <inertia
-	  ixx="0.1" ixy="0" ixz="0"
-	  iyy="0.1" iyz="0"
-	  izz="0.1"
+      <mass value="1.0"/>
+      <origin xyz="0.0 0 0" rpy=" 0 0 0"/>
+      <inertia
+        ixx="0.1" ixy="0" ixz="0"
+        iyy="0.1" iyz="0"
+        izz="0.1"
       />
     </inertial>
@@ -96,10 +91,22 @@
     </visual>
    </link>
-    <joint type="fixed" name="camera_plate_joint">
-    <origin xyz="0 0 0.3" rpy="0 0 0"/>
-    <child link="camera_plate"/>
-    <parent link="chassis"/>
-    <axis xyz="0 1 0" rpy="0 0 0"/>
-  </joint>
+    <joint type="continuous" name="camera_platform_joint">
+    <dynamics friction='.05'/>
+    <origin xyz="0 0 0.225" rpy="0 0 0"/>
+      <limit effort="30" velocity="1.0"/>
+    <child link="camera_platform"/>
+    <parent link="chassis"/>
+    <axis xyz="0 0 1" rpy="0 0 0"/>
+  </joint>
+  <transmission name="camera_platformtransmission">
+    <type>transmission_interface/SimpleTransmission</type>
+    <joint name="camera_platform_joint">
+      <hardwareInterface>hardware_interface/EffortJointInterface</hardwareInterface>
+    </joint>
+    <actuator name="camera_platform_joint">
+      <hardwareInterface>EffortJointInterface</hardwareInterface>
+      <mechanicalReduction>1</mechanicalReduction>
+    </actuator>
+  </transmission>
    <!-- Camera -->
     <link name="camera">
@@ -127,10 +134,41 @@
   </gazebo>
   <joint type="fixed" name="camera_joint">
-    <origin xyz="0.12 0 0" rpy="0 0 0"/>
+    <origin xyz="0.13 0 0" rpy="0 0 0"/>
     <child link="camera"/>
-    <parent link="camera_plate"/>
-    <axis xyz="0 1 0" rpy="0 0 0"/>
-  </joint>
-   <!-- Lidar -->
+    <parent link="camera_platform"/>
+    <axis xyz="0 0 0" rpy="0 0 0"/>
+  </joint>
+   <!-- Lidar platform -->
+  <link name="lidar_platform">
+    <pose>0 0 0 0 0 0</pose>
+    <inertial>
+      <mass value="1.0"/>
+      <origin xyz="0.0 0 0" rpy=" 0 0 0"/>
+      <inertia
+	  ixx="0.1" ixy="0" ixz="0"
+	  iyy="0.1" iyz="0"
+	  izz="0.1"
+      />
+    </inertial>
+    <collision name='collision'>
+      <origin xyz="0 0 0" rpy=" 0 0 0"/>
+      <geometry>
+      <cylinder length="0.05" radius="0.1"/>
+      </geometry>
+    </collision>
+    <visual>
+      <origin xyz="0 0 0" rpy=" 0 0 0"/>
+      <geometry>
+      <cylinder length="0.05" radius="0.1"/>
+      </geometry>
+    </visual>
+  </link>
+    <joint type="fixed" name="lidar_platform_join">
+    <origin xyz="0 0 0.3" rpy="0 0 0"/>
+    <child link="lidar_platform"/>
+    <parent link="chassis"/>
+    <axis xyz="0 1 0" rpy="0 0 0"/>
+  </joint>
+ <!-- Lidar -->
     <link name="hokuyo">
       <inertial>
@@ -154,7 +192,7 @@
     </link>
   <joint type="fixed" name="hokuyo_joint">
-    <origin xyz="0.15 0 0.15" rpy="0 0 0"/>
+    <origin xyz="0 0 0.05" rpy="0 0 0"/>
     <child link="hokuyo"/>
-    <parent link="chassis"/>
+    <parent link="lidar_platform"/>
     <axis xyz="0 1 0" rpy="0 0 0"/>
   </joint>
@@ -215,6 +253,3 @@
     </visual>
   </link>
-    <gazebo reference="chassis">
-    <material>Gazebo/Orange</material>
-  </gazebo>
 </robot>

Commit message: sensor upgrade RGB camera to Kinect camera

File: src/my_robot/urdf/my_robot.xacro (robot description, xacro)
@@ -110,5 +110,5 @@
   </transmission>
    <!-- Camera -->
-    <link name="camera">
+  <link name="camera">
       <inertial>
       <mass value="0.1"/>
@@ -129,8 +129,7 @@
 	  </geometry>
 	</visual>
-    </link>
-  <gazebo reference="camera">
-    <material>Gazebo/Red</material>
-  </gazebo>
+  </link>
+  <link name="camera_link_optical">
+  </link>
   <joint type="fixed" name="camera_joint">
     <origin xyz="0.13 0 0" rpy="0 0 0"/>
@@ -138,4 +137,9 @@
     <parent link="camera_platform"/>
     <axis xyz="0 0 0" rpy="0 0 0"/>
+  </joint>
+   <joint name="camera_optical_joint" type="fixed">
+    <origin xyz="0 0 0" rpy="-1.5707 0 -1.5707"/>
+    <parent link="camera"/>
+    <child link="camera_link_optical"/>
   </joint>
    <!-- Lidar platform -->
